File: hw/v1.sch (EAGLE design)
At the start: 44 parts, among them J1 FFC2B28-24-G, J2 S2B-PH-SM4-TB(LF)(SN), J3 10118193-0001LF, Q1 SI1308EDL-T1-GE3, U1 ESP32-C3-WROOM-02-H4, U2 PCF85063ATT/AJ, U3 TLV1117LV33DCYR, U4 MCP73831T-2ACI/OT, U5 MCP9700T-E/TT

Commit message: Hw changes
Parts:
- removed UART: 22-23-2041, con-molex:22-23-2041
- added J4: 851-43-004-20-001000, 851-43-004-20-001000:851-43-004-20-001000
- added LED2: (no value), led:LEDCHIP-LED0603
- added R11: 120, rcl:R-US_R0603
- added R12: 100k, rcl:R-US_R0603
Connections:
- new net DEBUG: R11.2, U1.IO5
- new net N$17: LED2.A, R11.1
- net 3V3: now also J4.4, R12.2; no longer UART-1.S
- net GND: now also J4.1, LED2.C; no longer UART-4.S
- net N$11: now also J4.3; no longer UART-2.S
- net N$12: now also J4.2; no longer UART-3.S
- net TEMP: now also R12.1
Other:
- moved on the sheet: C7, C8, C9, D1, D2, D3, L1, Q1, R1, R2
